File: CompressorNode.kicad_pcb (KiCad board)
At the start: 2 copper layers, 129.5 x 85.1 mm, 34 parts, among them J1 EXT1, J10 Screw_Terminal_01x03, J11 Screw_Terminal_01x02, J12 Screw_Terminal_01x03, J13 Screw_Terminal_01x04, J2 Screw_Terminal_01x04, J3 Screw_Terminal_01x03, J4 EXT2, J5 Screw_Terminal_01x02, J6 Screw_Terminal_01x02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

Commit message: Pressure sensor now connected to +5V instead of +3.3V
Connections:
- J12 pad 1: +3V3 -> +5V
Routing:
- net +5V: track 93.7 -> 135.6 mm
- net +3V3: track 135.2 -> 118.1 mm
Other:
- board text added: "Compressor/Laser cutter Node V0.12 Concept 2020 Makerspace Leiden"
- board text removed: "Compressor/Laser cutter Node V0.11 Concept 2020 Makerspace Leiden"
Changed lines of the file:
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@@
     (thickness 1.6)
     (drawings 59)
-    (tracks 176)
+    (tracks 174)
     (zones 0)
     (modules 34)
@@
     (title CompressorNode)
     (date 2020-04-02)
-    (rev "V0.11 Concept")
+    (rev "V0.12 Concept")
     (company "MakerSpace Leiden")
     (comment 1 "Getekend door Hans Beerman")
@@
   )
   (setup
-    (last_trace_width 1)
+    (last_trace_width 2)
     (user_trace_width 0.5)
     (user_trace_width 0.75)
@@
       (net 27 "Net-(J12-Pad2)"))
     (pad 1 thru_hole rect (at 0 0 180) (size 2.5 2.5) (drill 1.3) (layers *.Cu *.Mask)
-      (net 7 +3V3))
+      (net 5 +5V))
     (model ${KISYS3DMOD}/TerminalBlock_RND.3dshapes/TerminalBlock_RND_205-00288_1x03_P5.08mm_Horizontal.wrl
       (at (xyz 0 0 0))
@@
     (effects (font (size 1.2 1.2) (thickness 0.3)))
   )
-  (gr_text "Compressor/Laser cutter Node\nV0.11 Concept 2020\nMakerspace Leiden" (at 190.5 124.46) (layer F.SilkS)
+  (gr_text "Compressor/Laser cutter Node\nV0.12 Concept 2020\nMakerspace Leiden" (at 190.5 124.46) (layer F.SilkS)
     (effects (font (size 1.7 1.7) (thickness 0.4)))
   )
@@
   (segment (start 168.51 65.17) (end 167.64 66.04) (width 2) (layer F.Cu) (net 5))
   (segment (start 175.305 65.17) (end 168.51 65.17) (width 2) (layer F.Cu) (net 5))
-  (segment (start 149.86 75.565) (end 149.86 73.025) (width 2) (layer F.Cu) (net 5))
-  (segment (start 156.845 66.04) (end 167.64 66.04) (width 2) (layer F.Cu) (net 5))
-  (segment (start 149.86 73.025) (end 156.845 66.04) (width 2) (layer F.Cu) (net 5))
   (segment (start 149.86 81.915) (end 149.86 75.565) (width 2) (layer F.Cu) (net 5))
   (segment (start 147.955 83.82) (end 149.86 81.915) (width 2) (layer F.Cu) (net 5))
@@
   (segment (start 156.845 113.665) (end 156.845 109.22) (width 2) (layer F.Cu) (net 5))
   (segment (start 156.845 109.22) (end 147.955 100.33) (width 2) (layer F.Cu) (net 5))
+  (segment (start 123.825 60.25) (end 123.825 63.5) (width 2) (layer F.Cu) (net 5))
+  (segment (start 158.115 62.23) (end 155.575 59.69) (width 2) (layer F.Cu) (net 5))
+  (segment (start 155.575 59.69) (end 124.385 59.69) (width 2) (layer F.Cu) (net 5))
+  (segment (start 124.385 59.69) (end 123.825 60.25) (width 2) (layer F.Cu) (net 5))
+  (segment (start 158.115 66.04) (end 158.115 62.23) (width 2) (layer F.Cu) (net 5))
+  (segment (start 149.86 74.295) (end 158.115 66.04) (width 2) (layer F.Cu) (net 5))
+  (segment (start 149.86 75.565) (end 149.86 74.295) (width 2) (layer F.Cu) (net 5))
+  (segment (start 158.115 66.04) (end 167.64 66.04) (width 2) (layer F.Cu) (net 5))
   (segment (start 99.695 69.215) (end 99.695 63.5) (width 1) (layer B.Cu) (net 6))
   (segment (start 106.045 75.565) (end 99.695 69.215) (width 1) (layer B.Cu) (net 6))
@@
   (segment (start 123.825 83.82) (end 123.825 86.995) (width 1) (layer F.Cu) (net 6))
   (segment (start 123.825 86.995) (end 125.73 88.9) (width 1) (layer F.Cu) (net 6))
-  (segment (start 123.825 60.25) (end 123.825 63.5) (width 2) (layer F.Cu) (net 7))
-  (segment (start 123.265 59.69) (end 123.825 60.25) (width 2) (layer F.Cu) (net 7))
-  (segment (start 104.775 63.5) (end 104.775 60.325) (width 2) (layer F.Cu) (net 7))
-  (segment (start 105.41 59.69) (end 123.265 59.69) (width 2) (layer F.Cu) (net 7))
-  (segment (start 104.775 60.325) (end 105.41 59.69) (width 2) (layer F.Cu) (net 7))
-  (segment (start 141.605 81.28) (end 141.605 83.82) (width 2) (layer F.Cu) (net 7))
-  (segment (start 135.89 75.565) (end 141.605 81.28) (width 2) (layer F.Cu) (net 7))
-  (segment (start 127 75.565) (end 135.89 75.565) (width 2) (layer F.Cu) (net 7))
-  (segment (start 123.825 63.5) (end 123.825 72.39) (width 2) (layer F.Cu) (net 7))
-  (segment (start 123.825 72.39) (end 127 75.565) (width 2) (layer F.Cu) (net 7))
   (segment (start 104.775 63.5) (end 104.775 130.175) (width 2) (layer F.Cu) (net 7))
   (segment (start 141.605 86.995) (end 141.605 83.82) (width 1) (layer F.Cu) (net 7))
   (segment (start 135.89 88.9) (end 139.7 88.9) (width 1) (layer F.Cu) (net 7))
   (segment (start 139.7 88.9) (end 141.605 86.995) (width 1) (layer F.Cu) (net 7))
+  (segment (start 141.605 81.28) (end 141.605 83.82) (width 2) (layer F.Cu) (net 7))
+  (segment (start 104.775 75.565) (end 135.89 75.565) (width 2) (layer F.Cu) (net 7))
+  (segment (start 135.89 75.565) (end 141.605 81.28) (width 2) (layer F.Cu) (net 7))
   (segment (start 128.905 133.35) (end 128.905 109.22) (width 1) (layer F.Cu) (net 8))
   (segment (start 127 135.255) (end 128.905 133.35) (width 1) (layer F.Cu) (net 8))
@@
     (polygon
       (pts
-        (xy 167.64 81.28) (xy 175.895 92.075) (xy 175.895 104.775) (xy 172.72 108.585) (xy 172.72 139.065)
+        (xy 167.64 89.535) (xy 175.895 93.98) (xy 175.895 104.14) (xy 172.72 106.68) (xy 172.72 139.065)
         (xy 91.44 139.065) (xy 91.44 55.245) (xy 167.64 55.245)
       )

Commit message: Changed +3.3V text for pressure sensor to +5V on PCB, version not changed (v0.12)
Other:
- board text added: "+5V"
Changed lines of the file:
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@@
   )
   (setup
-    (last_trace_width 2)
+    (last_trace_width 0.25)
     (user_trace_width 0.5)
     (user_trace_width 0.75)
@@
       (padsonsilk false)
       (subtractmaskfromsilk false)
-      (outputformat 1)
+      (outputformat 4)
       (mirror false)
-      (drillshape 1)
+      (drillshape 0)
       (scaleselection 1)
       (outputdirectory ""))
@@
     (add_net +3V3)
     (add_net +5V)
-    (add_net ESP_EN)
     (add_net GND)
-    (add_net GPI34_BUT1)
     (add_net GPI35)
     (add_net GPI36_U1RXD)
     (add_net GPI39)
-    (add_net GPIO0)
     (add_net GPIO13_I2C-SDA)
     (add_net GPIO14_HS2_CLK)
     (add_net GPIO15_HS2_CMD)
     (add_net GPIO16_I2C-SCL)
-    (add_net GPIO1_U0TXD)
-    (add_net GPIO2_HS2_DATA0)
     (add_net GPIO32)
     (add_net GPIO33)
-    (add_net GPIO3_U0RXD)
     (add_net GPIO4_U1TXD)
     (add_net GPIO5_SPI_C5)
@@
     (effects (font (size 1.2 1.2) (thickness 0.3)))
   )
-  (gr_text +3.3V (at 113.03 71.12) (layer F.SilkS)
+  (gr_text +5V (at 113.03 71.12) (layer F.SilkS)
     (effects (font (size 1.2 1.2) (thickness 0.3)))
   )
